File: PhonoPreamp.kicad_sch (KiCad schematic)
At the start: 0 parts

Commit message: Main project
Added new schematic sheets.
Updated main project.
Other:
- added sheet Power (Power.kicad_sch)
- added sheet Preamp (Preamp.kicad_sch)
Changed lines of the file:
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@@
 		(company "Chapuzas S.L.")
+	)
+	(sheet
+		(at 158.75 67.31)
+		(size 92.71 52.07)
+		(exclude_from_sim no)
+		(in_bom yes)
+		(on_board yes)
+		(dnp no)
+		(fields_autoplaced yes)
+		(stroke
+			(width 0.1524)
+			(type solid)
+		)
+		(fill
+			(color 0 0 0 0.0000)
+		)
+		(property "Sheetname" "Power"
+			(at 158.75 66.5984 0)
+			(effects
+				(font
+					(size 1.27 1.27)
+				)
+				(justify left bottom)
+			)
+		)
+		(property "Sheetfile" "Power.kicad_sch"
+			(at 158.75 119.9646 0)
+			(effects
+				(font
+					(size 1.27 1.27)
+				)
+				(justify left top)
+			)
+		)
+		(instances
+			(project "PhonoPreamp"
+				(path "/7e93146b-7f37-4f4c-90dc-1ca52f83de10"
+					(page "2")
+				)
+			)
+		)
+	)
+	(sheet
+		(at 45.72 67.31)
+		(size 92.71 52.07)
+		(exclude_from_sim no)
+		(in_bom yes)
+		(on_board yes)
+		(dnp no)
+		(fields_autoplaced yes)
+		(stroke
+			(width 0.1524)
+			(type solid)
+		)
+		(fill
+			(color 0 0 0 0.0000)
+		)
+		(property "Sheetname" "Preamp"
+			(at 45.72 66.5984 0)
+			(effects
+				(font
+					(size 1.27 1.27)
+				)
+				(justify left bottom)
+			)
+		)
+		(property "Sheetfile" "Preamp.kicad_sch"
+			(at 45.72 119.9646 0)
+			(effects
+				(font
+					(size 1.27 1.27)
+				)
+				(justify left top)
+			)
+		)
+		(instances
+			(project "PhonoPreamp"
+				(path "/7e93146b-7f37-4f4c-90dc-1ca52f83de10"
+					(page "3")
+				)
+			)
+		)
 	)
 	(sheet_instances
