File: PhonoPreamp.kicad_pcb (KiCad board)
At the start: 2 copper layers, 0 parts

Commit message: Power Supply
Added the power supply board.
Parts:
- added C1: 2200u, Capacitor_SMD:CP_Elec_16x17.5, F.Cu at (94.0, 116.0)
- added C2: 2200u, Capacitor_SMD:CP_Elec_16x17.5, F.Cu at (94.0, 83.0)
- added C3: 2u2, Capacitor_SMD:CP_Elec_4x5.4, F.Cu at (105.0, 109.0)
- added C4: 2u2, Capacitor_SMD:CP_Elec_4x5.4, F.Cu at (107.0, 97.0)
- added C5: 2u2, Capacitor_SMD:CP_Elec_4x5.4, F.Cu at (111.0, 108.8)
- added C6: 2u2, Capacitor_SMD:CP_Elec_4x5.4, F.Cu at (108.0, 78.2)
- added C7: 100u, Capacitor_SMD:CP_Elec_6.3x7.7, F.Cu at (118.5, 113.3)
- added C8: 100u, Capacitor_SMD:CP_Elec_6.3x7.7, F.Cu at (115.0, 79.2)
- added D1: MDB6S, Custom_Parts:TSSOP-4_4.4x5mm_P4mm, F.Cu at (91.0, 100.0)
- added J1: Conn_01x01_Socket, Connector_Wire:SolderWire-2.5sqmm_1x01_D2.4mm_OD4.4mm, F.Cu at (30.5, 86.0)
- added J2: Conn_01x01_Socket, Connector_Wire:SolderWire-2.5sqmm_1x01_D2.4mm_OD4.4mm, F.Cu at (30.5, 113.0)
- added J3: Conn_01x03_Pin, Connector_Molex:Molex_KK-254_AE-6410-03A_1x03_P2.54mm_Vertical, F.Cu at (118.5, 98.2)
- added R1: 1K91, Resistor_SMD:R_0805_2012Metric_Pad1.20x1.40mm_HandSolder, F.Cu at (115.0, 119.5)
- added R2: 1K91, Resistor_SMD:R_0805_2012Metric_Pad1.20x1.40mm_HandSolder, F.Cu at (114.0, 87.0)
- added R3: 220, Resistor_SMD:R_0805_2012Metric_Pad1.20x1.40mm_HandSolder, F.Cu at (111.0, 113.5)
- added R4: 220, Resistor_SMD:R_0805_2012Metric_Pad1.20x1.40mm_HandSolder, F.Cu at (109.0, 83.2)
- added TR1: TEZ10.0-D-2, Transformer_THT:Transformer_Breve_TEZ-44x52, F.Cu at (47.0, 87.0)
- added U1: LM317_SOT-223, Package_TO_SOT_SMD:SOT-223-3_TabPin2, F.Cu at (109.8, 120.0)
- added U2: LM337_SOT223, Package_TO_SOT_SMD:SOT-223-3_TabPin2, F.Cu at (109.0, 89.5)
Routing:
- net Net-(D1--): track 0.00 -> 31.3 mm
- net +12V: track 0.00 -> 27.2 mm
- net Net-(D1-+): track 0.00 -> 26.4 mm
- net Net-(D1-Pad3): track 0.00 -> 18.1 mm
- net -12V: track 0.00 -> 17.8 mm
- net Net-(D1-Pad4): track 0.00 -> 17.7 mm
- net Net-(U1-ADJ): track 0.00 -> 6.90 mm
- net Net-(U2-ADJ): track 0.00 -> 6.46 mm
- net GND: vias 0 -> 85
- added copper zone on F.Cu, net -12V
- added copper zone on B.Cu, net GND
- added copper zone on F.Cu, net GND
- added copper zone on F.Cu, net Net-(J1-Pin_1)
- added copper zone on F.Cu, net Net-(J2-Pin_1)
Other:
- board outline added: 96.5 x 57 mm
