File: Preamp.kicad_sch (KiCad schematic)
At the start: 0 parts

Commit message: Preamp Schematic
Added the preamplifier schematic.
Parts:
- added C10, C11, C12, C13, C14, C40, C41, C43, C44, C9: 100n, Capacitor_SMD:C_0805_2012Metric_Pad1.18x1.45mm_HandSolder, symbol Device:C
- added C15, C26, C30, C47: 100p, Capacitor_SMD:C_0805_2012Metric_Pad1.18x1.45mm_HandSolder, symbol Device:C
- added C16, C21, C22, C23, C31, C35, C36, C37: 1u, Capacitor_SMD:C_0805_2012Metric_Pad1.18x1.45mm_HandSolder, symbol Device:C
- added C17, C18, C28, C29, C34, C48: 220u, Capacitor_SMD:CP_Elec_8x10, symbol Device:C_Polarized
- added C19, C32: 14.321n, Capacitor_SMD:C_0805_2012Metric_Pad1.18x1.45mm_HandSolder, symbol Device:C
- added C20, C33: 50n, Capacitor_SMD:C_0805_2012Metric_Pad1.18x1.45mm_HandSolder, symbol Device:C
- added C24, C42: 2u2, Capacitor_SMD:C_0805_2012Metric_Pad1.18x1.45mm_HandSolder, symbol Device:C
- added C25, C45: 2n2, Capacitor_SMD:C_0805_2012Metric_Pad1.18x1.45mm_HandSolder, symbol Device:C
- added C27, C46: 0u1, Capacitor_SMD:C_0805_2012Metric_Pad1.18x1.45mm_HandSolder, symbol Device:C
- added J10, J6: RCA in -, Connector_Wire:SolderWire-0.5sqmm_1x01_D0.9mm_OD2.1mm, symbol Connector:Conn_01x01_Socket
- added J12, J7: RCA out +, Connector_Wire:SolderWire-0.5sqmm_1x01_D0.9mm_OD2.1mm, symbol Connector:Conn_01x01_Socket
- added J13, J8: RCA out -, Connector_Wire:SolderWire-0.5sqmm_1x01_D0.9mm_OD2.1mm, symbol Connector:Conn_01x01_Socket
- added J4: Conn_01x03_Pin, Connector_Molex:Molex_KK-254_AE-6410-03A_1x03_P2.54mm_Vertical, symbol Connector:Conn_01x03_Pin
- added J5, J9: RCA in +, Connector_Wire:SolderWire-0.5sqmm_1x01_D0.9mm_OD2.1mm, symbol Connector:Conn_01x01_Socket
- added R10, R30: 4k22, Resistor_SMD:R_0805_2012Metric_Pad1.20x1.40mm_HandSolder, symbol Device:R
- added R11, R27, R32, R5: 221, Resistor_SMD:R_0805_2012Metric_Pad1.20x1.40mm_HandSolder, symbol Device:R
- added R12, R31: 5k23, Resistor_SMD:R_0805_2012Metric_Pad1.20x1.40mm_HandSolder, symbol Device:R
- added R13, R33: 63k4, Resistor_SMD:R_0805_2012Metric_Pad1.20x1.40mm_HandSolder, symbol Device:R
- added R14, R25: 150k, Resistor_SMD:R_0805_2012Metric_Pad1.20x1.40mm_HandSolder, symbol Device:R
- added R15, R34: 8k06, Resistor_SMD:R_0805_2012Metric_Pad1.20x1.40mm_HandSolder, symbol Device:R
- added R16, R36: 31k6, Resistor_SMD:R_0805_2012Metric_Pad1.20x1.40mm_HandSolder, symbol Device:R
- added R17, R35: 5k62, Resistor_SMD:R_0805_2012Metric_Pad1.20x1.40mm_HandSolder, symbol Device:R
- added R18, R37: 1k18, Resistor_SMD:R_0805_2012Metric_Pad1.20x1.40mm_HandSolder, symbol Device:R
- added R19, R38: 23k2, Resistor_SMD:R_0805_2012Metric_Pad1.20x1.40mm_HandSolder, symbol Device:R
- added R20, R39: 24k9, Resistor_SMD:R_0805_2012Metric_Pad1.20x1.40mm_HandSolder, symbol Device:R
- added R21, R41: 4K, Resistor_SMD:R_0805_2012Metric_Pad1.20x1.40mm_HandSolder, symbol Device:R
- added R22, R40: 0, Resistor_SMD:R_0805_2012Metric_Pad1.20x1.40mm_HandSolder, symbol Device:R
- added R23, R42: 1K, Resistor_SMD:R_0805_2012Metric_Pad1.20x1.40mm_HandSolder, symbol Device:R
- added R24, R7: 1M, Resistor_SMD:R_0805_2012Metric_Pad1.20x1.40mm_HandSolder, symbol Device:R
- added R26, R28, R8, R9: 2k, Resistor_SMD:R_0805_2012Metric_Pad1.20x1.40mm_HandSolder, symbol Device:R
- added R29, R6: 68k1, Resistor_SMD:R_0805_2012Metric_Pad1.20x1.40mm_HandSolder, symbol Device:R
- added U3, U4, U5, U6, U8: OPA1612AxD, Package_SO:SOIC-8_3.9x4.9mm_P1.27mm, symbol Amplifier_Operational:OPA1612AxD
Connections:
- new net: R28.1, R30.2, U6.7
- new net: R26.1, R28.2, U6.2 (-)
- new net: C19.2, C20.1, R12.1, R13.2
- new net: C19.1, R12.2, R5.2, U3.3 (+), U4.5 (+)
- new net: J12.1 (Pin_1), R42.1
- new net: C32.1, R27.2, R31.2, U3.5 (+), U6.5 (+)
- new net: C32.2, C33.1, R31.1, R33.2
- new net: C25.1, R18.1, R19.2, U5.5 (+)
- new net: C29.1, R27.1
- new net: R24.2, R26.2, U6.1
- new net: R30.1, R32.2, U6.6 (-)
- new net: C43.2, U8.4 (V-)
- new net: C44.1, U8.8 (V+)
- new net: C46.2, R39.1, R40.2, R41.1
- new net: C46.1, C47.1, R39.2, U8.6 (-)
- new net: C22.2, C23.1, R17.1
- new net: C24.1, R17.2, U5.1, U5.2 (-)
- new net: C35.2, C36.1, R34.2
- new net: C36.2, C37.1, R35.1
- new net: C30.1, C31.1, J9.1 (Pin_1), R25.2
- new net: C24.2, R18.2
- new net: C26.1, C27.1, R20.2, U5.6 (-)
- new net: C26.2, R22.1, R23.2, U5.7
- new net: C28.1, R21.2
- new net: C34.1, R32.1
- new net: C42.1, R35.2, U8.1, U8.2 (-)
- new net: C42.2, R37.2
- new net: C40.2, U6.4 (V-)
- new net: C41.1, U6.8 (V+)
- new net: C37.2, R36.2, U8.3 (+)
- new net: C33.2, C35.1, R33.1, U3.7
- new net: C48.1, R41.2
- new net: C27.2, R20.1, R21.1, R22.2
- new net: C23.2, R16.2, U5.3 (+)
- new net: R10.2, R9.1, U4.7
- new net: R8.1, R9.2, U4.2 (-)
- new net: C12.2, U5.4 (V-)
- new net: C18.1, R11.1
- new net: R10.1, R11.2, U4.6 (-)
- new net: C31.2, R24.1, R29.2, U3.6 (-)
- new net: J7.1 (Pin_1), R23.1
- new net: C14.2, U3.4 (V-)
- new net: C17.1, R5.1
- new net: C11.1, U5.8 (V+)
- new net: C13.2, U4.4 (V-)
- new net: C45.1, R37.1, R38.2, U8.5 (+)
- new net: C15.1, C16.1, J5.1 (Pin_1), R14.2
- new net: C20.2, C21.1, R13.1, U3.1
- new net: C21.2, C22.1, R15.2
- new net: C47.2, R40.1, R42.2, U8.7
- new net: R7.2, R8.2, U4.1
- new net: C9.1, U3.8 (V+)
- new net: C10.1, U4.8 (V+)
- new net: C16.2, R6.2, R7.1, U3.2 (-)
- new net +12V: C10.2, C11.2, C41.2, C44.2, C9.2, J4.3 (Pin_3)
- new net -12V: C12.1, C13.1, C14.1, C40.1, C43.1, J4.1 (Pin_1)
- new net GND: C15.2, C17.2, C18.2, C25.2, C28.2, C29.2, C30.2, C34.2, C45.2, C48.2, J10.1 (Pin_1), J13.1 (Pin_1), J6.1 (Pin_1), J8.1 (Pin_1), R14.1, R15.1, R16.1, R19.1, R25.1, R29.1, R34.1, R36.1, R38.1, R6.1, U4.3 (+), U6.3 (+)
