File: PowerSupply/PowerSupply.kicad_pcb (KiCad board)
At the start: 2 copper layers, 90 x 46 mm, 27 parts, among them J1 AC+, J2 AC-, J3 POWER, U1 LM317_SOT-223, U2 LM337_SOT223

Commit message: Power Supply Design
Updated the power supply schematic.
Updated the power supply board design.
Set the power supply project version to 1.1.
Parts:
- added C5: 10u, Capacitor_SMD:C_0805_2012Metric_Pad1.18x1.45mm_HandSolder, F.Cu at (177.2, 117.5)
- added C6: 10u, Capacitor_SMD:C_0805_2012Metric_Pad1.18x1.45mm_HandSolder, F.Cu at (177.2, 82.5)
- added D4: 1N4001, Diode_SMD:D_SOD-323, F.Cu at (177.9, 114.2)
- added D5: 1N4001, Diode_SMD:D_SOD-323, F.Cu at (177.9, 85.8)
- moved C10 0.75 mm to (180.8, 90.5)
- moved C9 0.75 mm to (180.8, 109.5)
- renumbered C8 to C10, C5 to C7, C6 to C8, C7 to C9
Routing:
- net -12V: track 5.35 -> 8.26 mm
- net +12V: track 11.2 -> 13.6 mm
- net Net-(D5-K): track 11.9 -> 9.94 mm
- net GND: vias 46 -> 44
- added copper zone on F.Cu, net Net-(D5-K)
Other:
- board text added: "V1.1"
- board text removed: "V1.0"
